Commit message: URDF of bot is created bot is moving with lidar map is not getting created

File: src/Agro_ros/urdf/robot.urdf (robot description, URDF)
Before this commit: robot Agrobot, 7 links, 6 joints
Links:
- removed link base_footprint
- removed link left_front_wheel
- removed link left_rare_wheel
- removed link lidar
- removed link right_front_wheel
- removed link right_rare_wheel
- added link track_outer_cover; visual mesh filename=package://Agro_ros/meshes/agro_ros_tracks_outer_cover.stl scale=0.05 0.05 0.05
- added link tracks; visual mesh filename=package://Agro_ros/meshes/agro_ros_tracks.stl scale=0.05 0.05 0.05
- added link water_level_sensor; visual mesh filename=package://Agro_ros/meshes/agro_ros_water_level_sensor.stl scale=0.05 0.05 0.05
- added link water_pump; visual mesh filename=package://Agro_ros/meshes/agro_ros_water_pump.stl scale=0.05 0.05 0.05
- link base_link: geometry visual mesh filename=package://Agro_ros/meshes/agro_ros_body.stl scale=0.05 0.05 0.05
Joints:
- removed joint base_footprint_joint
- removed joint base_left_front_wheel_joint
- removed joint base_left_rare_wheel_joint
- removed joint base_lidar_joint
- removed joint base_right_front_wheel_joint
- removed joint base_right_rare_wheel_joint
- added joint base_tracks_joint: type fixed, parent base_link, child tracks, origin xyz=0 0 0 rpy=0 0 0
- added joint base_tracks_outer_cover_joint: type fixed, parent base_link, child track_outer_cover, origin xyz=0 0 0 rpy=0 0 0
- added joint base_water_level_sensor_joint: type fixed, parent base_link, child water_level_sensor, origin xyz=0 0 0 rpy=0 0 0
- added joint base_water_pump_joint: type fixed, parent base_link, child water_pump, origin xyz=0 0 0 rpy=0 0 0

Commit message: now work with raspi as well as with the raspi with urdf, laser scan and mapping

File: src/Agro_ros/urdf/robot.urdf (robot description, URDF)
Before this commit: robot Agrobot, 5 links, 4 joints
Links:
- link base_link: geometry visual mesh filename=package://Agro_ros/meshes/agro_ros_body.stl scale=0.025 0.025 0.025
- link track_outer_cover: geometry visual mesh filename=package://Agro_ros/meshes/agro_ros_tracks_outer_cover.stl scale=0.025 0.025 0.025
- link tracks: geometry visual mesh filename=package://Agro_ros/meshes/agro_ros_tracks.stl scale=0.025 0.025 0.025
- link water_level_sensor: geometry visual mesh filename=package://Agro_ros/meshes/agro_ros_water_level_sensor.stl scale=0.025 0.025 0.025
- link water_pump: geometry visual mesh filename=package://Agro_ros/meshes/agro_ros_water_pump.stl scale=0.025 0.025 0.025
